File: 2502Tester/2502Tester.kicad_pcb (KiCad board)
At the start: 2 copper layers, 70 x 55 mm, 14 parts, among them J1_STEPPER1 STEPPER, J2_SERVO1 SERVO, J7 LeoPins8, J8 LeoPins0, J9 Leo_Power, SW1 SW_SERVO, SW2 SW_STEPPER

Commit message: Fix power pins offset by 1 pin
Parts:
- J7, J8, J9: moved to F.Cu
- moved J7 17.8 mm to (103.8, 69.4)
- moved J8 17.8 mm to (125.5, 69.4)
- moved J9 15.4 mm to (112.7, 117.6)
- moved C1 5.96 mm to (136.0, 114.4)
Routing:
- net +5V: track 41.5 -> 40.4 mm
- net /VIN: track 61.1 -> 61.7 mm

Commit message: Update board for fabrication v2
Parts:
- moved J8 0.09 mm to (125.6, 69.4)
Connections:
- J9 pad 1: unconnected-(J9-Pin_1-Pad1) -> (no net)
- J9 pad 2: unconnected-(J9-Pin_2-Pad2) -> (no net)
Other:
- board text added: "Arduino Leonardo Servo and Stepper Tester v2 Designed by X.Hunt 2026"
- board text removed: "3.3V"
- board text removed: "Arduino Leonardo Servo and Stepper Tester Designed by X.Hunt 2026"
